File: medreminder.kicad_pcb (KiCad board)
At the start: 2 copper layers, 60 x 28 mm, 11 parts, among them J3 LEDS, J4 USB_C_Receptacle_PowerOnly_6P, U1 XIAO-ESP32-C6, U2 ESP-12F

Commit message: all updates
Parts:
- added C1: 10uF, Capacitor_SMD:CP_Elec_4x5.4, F.Cu at (160.5, 115.9)
- added C2: 10uF, Capacitor_SMD:CP_Elec_4x5.4, F.Cu at (160.5, 121.8)
- added C3: 100nF, Capacitor_SMD:CP_Elec_4x5.4, F.Cu at (160.5, 127.6)
- added J1: USB_C PWR XIAO (SNAP), Connector_USB:USB_C_Receptacle_GCT_USB4135-GF-A_6P_TopMnt_Horizontal, F.Cu at (149.6, 117.7)
- added J2: USB_C PWR ESP-12F (SNAP), Connector_USB:USB_C_Receptacle_GCT_USB4135-GF-A_6P_TopMnt_Horizontal, F.Cu at (149.6, 127.0)
- added J5: LEDS, Connector_JST:JST_XH_B3B-XH-AM_1x03_P2.50mm_Vertical, F.Cu at (160.1, 133.9)
- added R11: 5.1k, Resistor_SMD:R_0603_1608Metric_Pad0.98x0.95mm_HandSolder, F.Cu at (149.8, 132.8)
- added R12: 5.1k, Resistor_SMD:R_0603_1608Metric_Pad0.98x0.95mm_HandSolder, F.Cu at (149.8, 135.3)
- added U3: XC6206PxxxMR, Package_TO_SOT_SMD:SOT-23-3, F.Cu at (145.1, 133.7)
- R4, R5, R6, R7, R8: value R_Small_US -> 10k
- U1: value XIAO-ESP32-C6 -> XIAO-ESP32-C6-SMD
Connections:
- R10 pad 2: Net-(J4-CC2) -> Net-(J2-CC2)
- R9 pad 1: Net-(J4-CC1) -> Net-(J2-CC1)

Commit message: V2 tabled
Parts:
- added J3_FFC_A1: FFC_CONN_12F, Connector_FFC-FPC:JUSHUO_AFA07-S06FCA-00_1x6-1MP_P1.0mm_Horizontal, F.Cu at (133.2, 80.0)
- added J4_FFC_B1: FFC_CONN_XIAO, Connector_FFC-FPC:JUSHUO_AFA07-S06FCA-00_1x6-1MP_P1.0mm_Horizontal, F.Cu at (116.5, 86.7)
- added J6: To USB-C (XIAO), Connector_PinHeader_2.54mm:PinHeader_1x02_P2.54mm_Vertical, F.Cu at (133.0, 120.5)
- added J7: TO USB-C (ESP), Connector_PinHeader_2.54mm:PinHeader_1x02_P2.54mm_Vertical, F.Cu at (94.5, 113.0)
- added REF**: MountingHole_3.2mm_M3, MountingHole:MountingHole_3.2mm_M3, F.Cu at (106.0, 125.5)
- added REF**: MouseBite-Slot_2.0x4.5mm_inset_D0.5mm_P0.85mm_7h, Panelization:MouseBite-Slot_2.0x4.5mm_inset_D0.5mm_P0.85mm_7h, F.Cu at (124.2, 86.8)
- added REF**: MouseBite-Slot_2.54x5.08mm_on-edge_D0.5mm_P0.85mm_5h_Trace, Panelization:MouseBite-Slot_2.54x5.08mm_on-edge_D0.5mm_P0.85mm_5h_Trace, F.Cu at (134.3, 118.0)
- added REF**: MouseBite-Slot_2.54x5.08mm_on-edge_D0.5mm_P0.85mm_5h_Trace, Panelization:MouseBite-Slot_2.54x5.08mm_on-edge_D0.5mm_P0.85mm_5h_Trace, F.Cu at (93.2, 118.0)
- C2: value 10uF -> 100nF
- C3: value 100nF -> 10uF
- J3: value LEDS -> TO ESP-12F; footprint Connector_JST:JST_XH_B3B-XH-AM_1x03_P2.50mm_Vertical -> Connector_PinHeader_2.54mm:PinHeader_1x02_P2.54mm_Vertical
- J4: value USB_C_Receptacle_PowerOnly_6P -> To XIAO; footprint Connector_USB:USB_C_Receptacle_GCT_USB4135-GF-A_6P_TopMnt_Horizontal -> Connector_PinHeader_2.54mm:PinHeader_1x02_P2.54mm_Vertical
- moved J3 80.2 mm to (94.5, 120.5), turned to -90 degrees
- moved C3 78.5 mm to (88.0, 97.5), turned to 90 degrees
- moved C2 74.4 mm to (88.0, 105.0), turned to 90 degrees
- moved R9 74.2 mm to (91.2, 123.5)
- moved R10 71.4 mm to (95.0, 123.5), turned to 180 degrees
- moved C1 61.8 mm to (99.2, 108.0)
- moved U3 58.3 mm to (93.0, 107.4), turned to -90 degrees
- moved J5 58.2 mm to (108.0, 108.0)
- moved J1 57.5 mm to (93.1, 128.5)
- moved J4 37.7 mm to (133.0, 113.0)
- moved R4 22.8 mm to (111.6, 99.8)
- moved R5 22.8 mm to (89.4, 88.0)
- moved R6 22.8 mm to (89.4, 91.5)
- moved R7 22.8 mm to (111.6, 97.8)
- moved R8 22.8 mm to (111.7, 95.8)
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Connections:
- C1 pad 2: Net-(U3-GND) -> GND
- C2 pad 2: Net-(U3-GND) -> GND
- C3 pad 2: Net-(U3-GND) -> GND
- R10 pad 2: Net-(J2-CC2) -> Net-(J1-CC2)
- R11 pad 1: Net-(J1-CC1) -> Net-(J2-CC1)
- R12 pad 2: Net-(J1-CC2) -> Net-(J2-CC2)
- R9 pad 1: Net-(J2-CC1) -> Net-(J1-CC1)
- U3 pad 1: Net-(U3-GND) -> GND
Routing:
- net +3.3V: track 61.6 -> 7.41 mm
- net /LED_DATA: track 40.0 -> 0.00 mm, vias 1 -> 0
- net +5V: track 12.4 -> 51.4 mm, vias 0 -> 2
- net /UART_RX: track 38.9 -> 13.4 mm
- net /UART_TX: track 13.6 -> 36.4 mm, vias 2 -> 0
- net GND: track 0.00 -> 15.7 mm, vias 15 -> 31
- net /RST: track 3.56 -> 0.00 mm
- net /EN: track 3.52 -> 0.00 mm
- net /GPIO0: track 2.97 -> 0.00 mm
- net /GPIO2: track 2.89 -> 0.00 mm
- net /GPIO15: track 2.89 -> 0.00 mm
- net Net-(J4-CC2): track 2.51 -> 0.00 mm
- net Net-(J4-CC1): track 2.51 -> 0.00 mm
- net Net-(J2-CC2): track 0.00 -> 2.46 mm
- net Net-(J2-CC1): track 0.00 -> 2.46 mm
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- added copper zone on F.Cu, net +3.3V
Other:
- board size 60 x 28 mm -> 66.5 x 57 mm
