File: medreminder.kicad_sch (KiCad schematic)
At the start: 11 parts, among them J3 LEDS, J4 USB_C_Receptacle_PowerOnly_6P, U1 XIAO-ESP32-C6-SMD, U2 ESP-12F

Commit message: all updates
Parts:
- added C1, C2: 10uF, Capacitor_SMD:CP_Elec_4x5.4, symbol Device:C_Polarized_Small_US
- added C3: 100nF, Capacitor_SMD:CP_Elec_4x5.4, symbol Device:C_Polarized_Small_US
- added J1: USB_C PWR XIAO (SNAP), Connector_USB:USB_C_Receptacle_GCT_USB4135-GF-A_6P_TopMnt_Horizontal, symbol Connector:USB_C_Receptacle_PowerOnly_6P
- added J3_FFC_A1: FFC_CONN_12F, symbol Connector_Generic:Conn_01x06
- added J4_FFC_B1: FFC_CONN_XIAO, symbol Connector_Generic:Conn_01x06
- added R11, R12: 5.1k, Resistor_SMD:R_0603_1608Metric_Pad0.98x0.95mm_HandSolder, symbol Device:R_Small_US
- added U3: XC6206PxxxMR, Package_TO_SOT_SMD:SOT-23-3, symbol Regulator_Linear:XC6206PxxxMR
- J2: renamed from J4; value USB_C_Receptacle_PowerOnly_6P -> USB_C PWR ESP-12F (SNAP)
- R4, R5, R6, R7, R8: value R_Small_US -> 10k
- renumbered J3 to J5
Connections:
- net +3.3V: now also C2.1, C3.1, J3_FFC_A1.3 (Pin_3), J4_FFC_B1.3 (Pin_3), U3.2 (VO)
- net +5V: now also C1.1, J1.A9 (VBUS), J1.B9 (VBUS), U3.3 (VI)
- net GND: now also J1.A12 (GND), J1.B12 (GND), J1.SH (SHIELD), J3_FFC_A1.1 (Pin_1), J3_FFC_A1.6 (Pin_6), J4_FFC_B1.1 (Pin_1), J4_FFC_B1.6 (Pin_6), R11.2, R12.1
- net UART_RX: now also J3_FFC_A1.2 (Pin_2), J4_FFC_B1.2 (Pin_2)
- net UART_TX: now also J3_FFC_A1.5 (Pin_5), J4_FFC_B1.5 (Pin_5)
- new net: C1.2, C2.2, C3.2, U3.1 (GND)
- new net: J1.B5 (CC2), R12.2
- new net: J1.A5 (CC1), R11.1
Other:
- note added: "ESP-12F sub-board"
- note added: "USB-C Power (SNAP)"
- note added: "XIAO sub-board"
- moved on the sheet: J2, J5, R10, R4, R5, R6, R7, R8, R9, U1, U2

Commit message: V2 tabled
Parts:
- added J3: TO ESP-12F, symbol Connector_Generic:Conn_01x02
- added J4: To XIAO, symbol Connector_Generic:Conn_01x02
- added J6: To USB-C, symbol Connector_Generic:Conn_01x02
- added J7: TO USB-C, symbol Connector_Generic:Conn_01x02
- J3_FFC_A1, J4_FFC_B1: footprint (none) -> Connector_FFC-FPC:JUSHUO_AFA07-S06FCA-00_1x6-1MP_P1.0mm_Horizontal
- renumbered C3 to C2, C2 to C3
Connections:
- net +5V: now also J3.1 (Pin_1), J4.1 (Pin_1), J6.1 (Pin_1), J7.1 (Pin_1)
- net GND: now also C1.2, C2.2, C3.2, U3.1 (GND), J3.2 (Pin_2), J4.2 (Pin_2), J6.2 (Pin_2), J7.2 (Pin_2)
Other:
- moved on the sheet: J1, J2, R10, R11, R12, R9
